File: Hardware/CC3000_WiFi_Breakout.sch (EAGLE design)
At the start: 33 parts, among them J1 U.FL, U1 V_REG_317SMD, U3 74HC4050, U5 CC3000

Commit message: Layout (mostly) done
Parts:
- U1: value V_REG_317SMD -> (none); device SparkFun-PowerIC:V_REG_317SMD -> SparkFun-PowerIC:V_REG_LM1117SOT223
Connections:
- net 3.3V: now also U1.OUT@1
Other:
- note added: "Breakout Header"
- note removed: "Arduino Headers"
- moved on the sheet: R1, R2
Changed lines of the file:
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@@
 <part name="R1" library="SparkFun-Resistors" deviceset="RESISTOR" device="0603" value="240"/>
 <part name="R2" library="SparkFun-Resistors" deviceset="RESISTOR" device="0603" value="390"/>
-<part name="U1" library="SparkFun-PowerIC" deviceset="V_REG_317" device="SMD"/>
+<part name="U1" library="SparkFun-PowerIC" deviceset="V_REG_LM1117" device="SOT223"/>
 <part name="GND1" library="SparkFun-Aesthetics" deviceset="GND" device=""/>
 <part name="GND2" library="SparkFun-Aesthetics" deviceset="GND" device=""/>
@@
 <text x="2.54" y="132.08" size="2.54" layer="97">Power</text>
 <text x="2.54" y="101.6" size="2.54" layer="97">Debug</text>
-<text x="2.54" y="50.8" size="2.54" layer="97">Arduino Headers</text>
+<text x="2.54" y="50.8" size="2.54" layer="97">Breakout Header</text>
 <text x="2.54" y="2.54" size="2.54" layer="97">Level Shifter</text>
 <text x="149.86" y="38.1" size="2.54" layer="97">WiFi</text>
@@
 <instance part="C3" gate="G$1" x="25.4" y="167.64"/>
 <instance part="C4" gate="G$1" x="71.12" y="167.64"/>
-<instance part="R1" gate="G$1" x="50.8" y="167.64" smashed="yes" rot="R90">
-<attribute name="NAME" x="53.34" y="170.1546" size="1.778" layer="95"/>
-<attribute name="VALUE" x="53.34" y="165.1" size="1.778" layer="96"/>
-</instance>
-<instance part="R2" gate="G$1" x="40.64" y="152.4" smashed="yes" rot="R90">
-<attribute name="NAME" x="43.18" y="154.9146" size="1.778" layer="95"/>
-<attribute name="VALUE" x="43.18" y="152.4" size="1.778" layer="96"/>
+<instance part="R1" gate="G$1" x="50.8" y="165.1" smashed="yes" rot="R90">
+<attribute name="NAME" x="53.34" y="167.6146" size="1.778" layer="95"/>
+<attribute name="VALUE" x="53.34" y="162.56" size="1.778" layer="96"/>
+</instance>
+<instance part="R2" gate="G$1" x="40.64" y="149.86" smashed="yes" rot="R90">
+<attribute name="NAME" x="43.18" y="152.3746" size="1.778" layer="95"/>
+<attribute name="VALUE" x="43.18" y="149.86" size="1.778" layer="96"/>
 </instance>
 <instance part="U1" gate="G$1" x="40.64" y="175.26" smashed="yes">
@@
 <attribute name="VALUE" x="35.56" y="179.07" size="1.778" layer="96"/>
 </instance>
-<instance part="GND1" gate="1" x="40.64" y="142.24"/>
-<instance part="GND2" gate="1" x="25.4" y="142.24"/>
-<instance part="GND3" gate="1" x="15.24" y="142.24"/>
-<instance part="GND4" gate="1" x="60.96" y="142.24"/>
-<instance part="GND5" gate="1" x="71.12" y="142.24"/>
+<instance part="GND1" gate="1" x="40.64" y="139.7"/>
+<instance part="GND2" gate="1" x="25.4" y="139.7"/>
+<instance part="GND3" gate="1" x="15.24" y="139.7"/>
+<instance part="GND4" gate="1" x="60.96" y="139.7"/>
+<instance part="GND5" gate="1" x="71.12" y="139.7"/>
 <instance part="U3" gate="G$1" x="40.64" y="20.32"/>
 <instance part="GND6" gate="1" x="60.96" y="30.48"/>
@@
 <attribute name="VALUE" x="86.36" y="167.64" size="1.778" layer="96"/>
 </instance>
-<instance part="GND19" gate="1" x="83.82" y="142.24"/>
+<instance part="GND19" gate="1" x="83.82" y="139.7"/>
 <instance part="D1" gate="G$1" x="83.82" y="157.48" smashed="yes">
 <attribute name="NAME" x="86.36" y="157.48" size="1.778" layer="95"/>
@@
 <pinref part="U1" gate="G$1" pin="ADJ"/>
 <pinref part="R2" gate="G$1" pin="2"/>
-<wire x1="40.64" y1="167.64" x2="40.64" y2="160.02" width="0.1524" layer="91"/>
+<wire x1="40.64" y1="167.64" x2="40.64" y2="157.48" width="0.1524" layer="91"/>
 <pinref part="R1" gate="G$1" pin="1"/>
-<wire x1="40.64" y1="160.02" x2="40.64" y2="157.48" width="0.1524" layer="91"/>
-<wire x1="50.8" y1="162.56" x2="50.8" y2="160.02" width="0.1524" layer="91"/>
-<wire x1="50.8" y1="160.02" x2="40.64" y2="160.02" width="0.1524" layer="91"/>
-<junction x="40.64" y="160.02"/>
+<wire x1="40.64" y1="157.48" x2="40.64" y2="154.94" width="0.1524" layer="91"/>
+<wire x1="50.8" y1="160.02" x2="50.8" y2="157.48" width="0.1524" layer="91"/>
+<wire x1="50.8" y1="157.48" x2="40.64" y2="157.48" width="0.1524" layer="91"/>
+<junction x="40.64" y="157.48"/>
 </segment>
 </net>
@@
 <wire x1="50.8" y1="175.26" x2="50.8" y2="172.72" width="0.1524" layer="91"/>
 <pinref part="C2" gate="G$1" pin="+"/>
+<wire x1="50.8" y1="172.72" x2="50.8" y2="170.18" width="0.1524" layer="91"/>
 <wire x1="50.8" y1="175.26" x2="60.96" y2="175.26" width="0.1524" layer="91"/>
 <wire x1="60.96" y1="175.26" x2="60.96" y2="172.72" width="0.1524" layer="91"/>
@@
 <wire x1="71.12" y1="172.72" x2="71.12" y2="175.26" width="0.1524" layer="91"/>
 <junction x="71.12" y="175.26"/>
+<pinref part="U1" gate="G$1" pin="OUT@1"/>
+<wire x1="48.26" y1="172.72" x2="50.8" y2="172.72" width="0.1524" layer="91"/>
+<junction x="50.8" y="172.72"/>
 </segment>
 <segment>
@@
 <pinref part="C1" gate="G$1" pin="-"/>
 <pinref part="GND3" gate="1" pin="GND"/>
-<wire x1="15.24" y1="165.1" x2="15.24" y2="144.78" width="0.1524" layer="91"/>
+<wire x1="15.24" y1="165.1" x2="15.24" y2="142.24" width="0.1524" layer="91"/>
 </segment>
 <segment>
 <pinref part="C3" gate="G$1" pin="2"/>
 <pinref part="GND2" gate="1" pin="GND"/>
-<wire x1="25.4" y1="165.1" x2="25.4" y2="144.78" width="0.1524" layer="91"/>
+<wire x1="25.4" y1="165.1" x2="25.4" y2="142.24" width="0.1524" layer="91"/>
 </segment>
 <segment>
 <pinref part="R2" gate="G$1" pin="1"/>
 <pinref part="GND1" gate="1" pin="GND"/>
-<wire x1="40.64" y1="147.32" x2="40.64" y2="144.78" width="0.1524" layer="91"/>
+<wire x1="40.64" y1="144.78" x2="40.64" y2="142.24" width="0.1524" layer="91"/>
 </segment>
 <segment>
 <pinref part="C2" gate="G$1" pin="-"/>
 <pinref part="GND4" gate="1" pin="GND"/>
-<wire x1="60.96" y1="165.1" x2="60.96" y2="144.78" width="0.1524" layer="91"/>
+<wire x1="60.96" y1="165.1" x2="60.96" y2="142.24" width="0.1524" layer="91"/>
 </segment>
 <segment>
 <pinref part="C4" gate="G$1" pin="2"/>
 <pinref part="GND5" gate="1" pin="GND"/>
-<wire x1="71.12" y1="165.1" x2="71.12" y2="144.78" width="0.1524" layer="91"/>
+<wire x1="71.12" y1="165.1" x2="71.12" y2="142.24" width="0.1524" layer="91"/>
 </segment>
 <segment>
@@
 <pinref part="D1" gate="G$1" pin="C"/>
 <pinref part="GND19" gate="1" pin="GND"/>
-<wire x1="83.82" y1="152.4" x2="83.82" y2="144.78" width="0.1524" layer="91"/>
-</segment>
-<segment>
+<wire x1="83.82" y1="152.4" x2="83.82" y2="142.24" width="0.1524" layer="91"/>
+</segment>
+<segment>

Commit message: Proto layout complete. Needs aesthetics.
Connections:
- net D4 renamed INT
- net D5 renamed CS
- removed net D1: JP2.1, U3.1A
- removed net D2: JP2.2, U3.2A
- removed net D3: JP2.3, U3.3A
- new net EN: JP2.2, U3.1A
- new net MOSI: JP2.7, U3.3A
- new net SCK: JP2.3, U3.2A
- net GND: now also JP2.1; no longer JP2.7
Changed lines of the file:
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@@
 <instance part="SUPPLY3" gate="1" x="73.66" y="73.66"/>
 <instance part="SUPPLY4" gate="1" x="15.24" y="177.8"/>
-<instance part="GND7" gate="1" x="58.42" y="66.04"/>
+<instance part="GND7" gate="1" x="53.34" y="91.44"/>
 <instance part="STANDOFF1" gate="G$1" x="233.68" y="33.02"/>
 <instance part="STANDOFF2" gate="G$1" x="228.6" y="33.02"/>
@@
 <segment>
 <pinref part="JP2" gate="G$1" pin="8"/>
-<wire x1="45.72" y1="68.58" x2="53.34" y2="68.58" width="0.1524" layer="91"/>
-<wire x1="53.34" y1="68.58" x2="53.34" y2="60.96" width="0.1524" layer="91"/>
 <pinref part="SUPPLY1" gate="G$1" pin="3.3V"/>
-<wire x1="53.34" y1="60.96" x2="66.04" y2="60.96" width="0.1524" layer="91"/>
-<wire x1="66.04" y1="60.96" x2="66.04" y2="73.66" width="0.1524" layer="91"/>
+<wire x1="45.72" y1="68.58" x2="66.04" y2="68.58" width="0.1524" layer="91"/>
+<wire x1="66.04" y1="68.58" x2="66.04" y2="73.66" width="0.1524" layer="91"/>
 </segment>
 </net>
@@
 </segment>
 <segment>
-<pinref part="JP2" gate="G$1" pin="7"/>
+<pinref part="JP2" gate="G$1" pin="1"/>
+<wire x1="45.72" y1="86.36" x2="48.26" y2="86.36" width="0.1524" layer="91"/>
+<wire x1="48.26" y1="86.36" x2="48.26" y2="96.52" width="0.1524" layer="91"/>
 <pinref part="GND7" gate="1" pin="GND"/>
-<wire x1="45.72" y1="71.12" x2="58.42" y2="71.12" width="0.1524" layer="91"/>
-<wire x1="58.42" y1="71.12" x2="58.42" y2="68.58" width="0.1524" layer="91"/>
+<wire x1="48.26" y1="96.52" x2="53.34" y2="96.52" width="0.1524" layer="91"/>
+<wire x1="53.34" y1="96.52" x2="53.34" y2="93.98" width="0.1524" layer="91"/>
 </segment>
 </net>
 <net name="WIFI_CS" class="0">
 <segment>
-<label x="76.2" y="25.4" size="1.27" layer="95" xref="yes"/>
 <pinref part="R4" gate="G$1" pin="1"/>
-<wire x1="71.12" y1="25.4" x2="76.2" y2="25.4" width="0.1524" layer="91"/>
-<wire x1="71.12" y1="27.94" x2="71.12" y2="25.4" width="0.1524" layer="91"/>
+<pinref part="U3" gate="G$1" pin="5Y"/>
+<wire x1="50.8" y1="15.24" x2="71.12" y2="15.24" width="0.1524" layer="91"/>
+<label x="76.2" y="15.24" size="1.27" layer="95" xref="yes"/>
+<wire x1="71.12" y1="15.24" x2="76.2" y2="15.24" width="0.1524" layer="91"/>
+<wire x1="71.12" y1="27.94" x2="71.12" y2="15.24" width="0.1524" layer="91"/>
+<junction x="71.12" y="15.24"/>
 </segment>
 <segment>
@@
 <wire x1="165.1" y1="68.58" x2="165.1" y2="63.5" width="0.1524" layer="91"/>
 <label x="165.1" y="63.5" size="1.27" layer="95" rot="R270" xref="yes"/>
-</segment>
-<segment>
-<pinref part="U3" gate="G$1" pin="5Y"/>
-<wire x1="50.8" y1="15.24" x2="55.88" y2="15.24" width="0.1524" layer="91"/>
-<label x="55.88" y="15.24" size="1.27" layer="95" xref="yes"/>
 </segment>
 </net>
@@
 <segment>
 <pinref part="JP2" gate="G$1" pin="9"/>
-<wire x1="45.72" y1="66.04" x2="50.8" y2="66.04" width="0.1524" layer="91"/>
-<wire x1="50.8" y1="66.04" x2="50.8" y2="58.42" width="0.1524" layer="91"/>
 <pinref part="SUPPLY3" gate="1" pin="VCC"/>
-<wire x1="50.8" y1="58.42" x2="73.66" y2="58.42" width="0.1524" layer="91"/>
-<wire x1="73.66" y1="58.42" x2="73.66" y2="73.66" width="0.1524" layer="91"/>
-</segment>
-</net>
-<net name="D1" class="0">
-<segment>
-<pinref part="U3" gate="G$1" pin="1A"/>
-<wire x1="30.48" y1="25.4" x2="25.4" y2="25.4" width="0.1524" layer="91"/>
-</segment>
-<segment>
-<pinref part="JP2" gate="G$1" pin="1"/>
-<wire x1="45.72" y1="86.36" x2="50.8" y2="86.36" width="0.1524" layer="91"/>
-<label x="50.8" y="86.36" size="1.27" layer="95" xref="yes"/>
-</segment>
-</net>
-<net name="D2" class="0">
-<segment>
-<pinref part="U3" gate="G$1" pin="2A"/>
-<wire x1="30.48" y1="22.86" x2="25.4" y2="22.86" width="0.1524" layer="91"/>
-</segment>
+<wire x1="45.72" y1="66.04" x2="73.66" y2="66.04" width="0.1524" layer="91"/>
+<wire x1="73.66" y1="66.04" x2="73.66" y2="73.66" width="0.1524" layer="91"/>
+</segment>
+</net>
+<net name="EN" class="0">
 <segment>
 <pinref part="JP2" gate="G$1" pin="2"/>
@@
 <label x="50.8" y="83.82" size="1.27" layer="95" xref="yes"/>
 </segment>
-</net>
-<net name="D3" class="0">
-<segment>
-<pinref part="U3" gate="G$1" pin="3A"/>
-<wire x1="30.48" y1="20.32" x2="25.4" y2="20.32" width="0.1524" layer="91"/>
-</segment>
+<segment>
+<pinref part="U3" gate="G$1" pin="1A"/>
+<wire x1="30.48" y1="25.4" x2="25.4" y2="25.4" width="0.1524" layer="91"/>
+<label x="25.4" y="25.4" size="1.27" layer="95" rot="R180" xref="yes"/>
+</segment>
+</net>
+<net name="SCK" class="0">
 <segment>
 <pinref part="JP2" gate="G$1" pin="3"/>
@@
 <label x="50.8" y="81.28" size="1.27" layer="95" xref="yes"/>
 </segment>
-</net>
-<net name="D4" class="0">
+<segment>
+<pinref part="U3" gate="G$1" pin="2A"/>
+<wire x1="30.48" y1="22.86" x2="25.4" y2="22.86" width="0.1524" layer="91"/>
+<label x="25.4" y="22.86" size="1.27" layer="95" rot="R180" xref="yes"/>
+</segment>
+</net>
+<net name="MOSI" class="0">
+<segment>
+<pinref part="JP2" gate="G$1" pin="7"/>
+<wire x1="45.72" y1="71.12" x2="50.8" y2="71.12" width="0.1524" layer="91"/>
+<label x="50.8" y="71.12" size="1.27" layer="95" xref="yes"/>
+</segment>
+<segment>
+<pinref part="U3" gate="G$1" pin="3A"/>
+<wire x1="30.48" y1="20.32" x2="25.4" y2="20.32" width="0.1524" layer="91"/>
+<label x="25.4" y="20.32" size="1.27" layer="95" rot="R180" xref="yes"/>
+</segment>
+</net>
+<net name="INT" class="0">
 <segment>
 <pinref part="U3" gate="G$1" pin="4A"/>
 <wire x1="30.48" y1="17.78" x2="25.4" y2="17.78" width="0.1524" layer="91"/>
+<label x="25.4" y="17.78" size="1.27" layer="95" rot="R180" xref="yes"/>
 </segment>
 <segment>
@@
 </segment>
 </net>
-<net name="D5" class="0">
+<net name="CS" class="0">
 <segment>
 <pinref part="U3" gate="G$1" pin="5A"/>
 <wire x1="30.48" y1="15.24" x2="25.4" y2="15.24" width="0.1524" layer="91"/>
-</segment>
-<segment>
+<label x="25.4" y="15.24" size="1.27" layer="95" rot="R180" xref="yes"/>
+</segment>
+<segment>

Commit message: Prototype board ready for review
Parts:
- U1: value (none) -> LM1117
Changed lines of the file:
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@@
 <setting verticaltext="up"/>
 </settings>
-<grid distance="0.1" unitdist="inch" unit="inch" style="lines" multiple="1" display="yes" altdistance="0.01" altunitdist="inch" altunit="inch"/>
+<grid distance="0.1" unitdist="inch" unit="inch" style="lines" multiple="1" display="no" altdistance="0.01" altunitdist="inch" altunit="inch"/>
 <layers>
 <layer number="1" name="Top" color="4" fill="1" visible="no" active="no"/>
@@
 <part name="R1" library="SparkFun-Resistors" deviceset="RESISTOR" device="0603" value="240"/>
 <part name="R2" library="SparkFun-Resistors" deviceset="RESISTOR" device="0603" value="390"/>
-<part name="U1" library="SparkFun-PowerIC" deviceset="V_REG_LM1117" device="SOT223"/>
+<part name="U1" library="SparkFun-PowerIC" deviceset="V_REG_LM1117" device="SOT223" value="LM1117"/>
 <part name="GND1" library="SparkFun-Aesthetics" deviceset="GND" device=""/>
 <part name="GND2" library="SparkFun-Aesthetics" deviceset="GND" device=""/>

Commit message: Ready for prototype
Changed lines of the file:
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@@
 <setting verticaltext="up"/>
 </settings>
-<grid distance="0.1" unitdist="inch" unit="inch" style="lines" multiple="1" display="no" altdistance="0.01" altunitdist="inch" altunit="inch"/>
+<grid distance="0.1" unitdist="inch" unit="inch" style="lines" multiple="1" display="yes" altdistance="0.01" altunitdist="inch" altunit="inch"/>
 <layers>
 <layer number="1" name="Top" color="4" fill="1" visible="no" active="no"/>
@@
 <sheet>
 <plain>
-<text x="172.72" y="7.62" size="5.08" layer="94">Shawn Hymel</text>
+<text x="172.72" y="12.7" size="2.54" layer="94" align="center-left">Shawn Hymel</text>
 <text x="237.236" y="6.604" size="3.81" layer="94">v01</text>
 <wire x1="0" y1="129.54" x2="101.6" y2="129.54" width="0.1524" layer="97" style="longdash"/>

Commit message: Changed layout for board
Parts:
- removed STANDOFF3, STANDOFF4: STAND-OFF, SparkFun-Electromechanical:STAND-OFF
- C1, C2: device SparkFun-Capacitors:CAP_POL1206 -> SparkFun-Capacitors:CAP0805
Connections:
- net CS renamed CS_5V
- net EN renamed EN_5V
- net MOSI renamed MOSI_5V
- net SCK renamed SCK_5V
- net SPI_MISO renamed MISO_3.3V
- net SPI_MOSI renamed MOSI_3.3V
- net SPI_SCK renamed SCK_3.3V
- net WIFI_CS renamed CS_3.3V
- net WIFI_EN renamed EN_3.3V
- removed net INT: JP2.4, U3.4A
- removed net WIFI_INT: U3.4Y, U5.SPI_IRQ
- new net INT_3.3V: JP2.4, U5.SPI_IRQ
- net 3.3V: now also C2.1; no longer C2.+
- net GND: now also C1.2, C2.2; no longer C1.-, C2.-
- net VCC: now also C1.1; no longer C1.+
Other:
- note added: "v02"
- note removed: "v01"

Commit message: Redid layout. Again.
Parts:
- removed LOGO2: LOGO-SFENEW, SparkFun-Aesthetics:LOGO-SFENEW
- added LOGO4: SFE_LOGO_NAME_FLAME.1_INCH, SparkFun-Aesthetics:SFE_LOGO_NAME_FLAME.1_INCH
Connections:
- net 3.3V: now also JP2.7; no longer JP2.8
- net CS_5V: now also JP2.4; no longer JP2.5
- net EN_5V: now also JP2.1; no longer JP2.2
- net GND: now also JP2.9; no longer JP2.1
- net INT_3.3V: now also JP2.3; no longer JP2.4
- net MISO_3.3V: now also JP2.5; no longer JP2.6
- net MOSI_5V: now also JP2.6; no longer JP2.7
- net SCK_5V: now also JP2.2; no longer JP2.3
- net VCC: now also JP2.8; no longer JP2.9
Other:
- moved on the sheet: AE1, C5, C6, C7, C8, J1, L1, L2, SJ1, U5
